Commit message: Updated URDF for accurate representation

File: src/mark_five_description/urdf/robot.urdf (robot description, URDF)
Before this commit: robot mark_five_robot, 4 links, 3 joints
Links:
- removed link lidar
- added link antenna_left_link; visual cylinder length=0.016 radius=0.006; visual cylinder length=0.150 radius=0.004
- added link antenna_right_link; visual cylinder length=0.016 radius=0.006; visual cylinder length=0.150 radius=0.004
- added link arduino_mega_link, mass 0.05; collision box size=0.101 0.053 0.015; visual box size=0.012 0.010 0.008
- added link base_footprint
- added link jetson_nano_link, mass 0.3; collision box size=0.100 0.080 0.050; visual box size=0.090 0.070 0.008
- added link left_front_sprocket; visual cylinder length=0.004 radius=0.028; visual cylinder length=0.004 radius=0.028
- added link left_idler; visual cylinder length=0.030 radius=0.018; visual cylinder length=0.035 radius=0.008
- added link left_motor_link; visual box size=0.024 0.024 0.020; visual cylinder length=0.012 radius=0.003
- added link left_rear_sprocket; visual cylinder length=0.004 radius=0.028; visual cylinder length=0.004 radius=0.028
- added link platform_link, mass 0.3; collision box size=0.220 0.200 0.003; visual box size=0.220 0.200 0.003
- added link right_front_sprocket; visual cylinder length=0.004 radius=0.028; visual cylinder length=0.004 radius=0.028
- added link right_idler; visual cylinder length=0.030 radius=0.018; visual cylinder length=0.035 radius=0.008
- added link right_motor_link; visual box size=0.024 0.024 0.020; visual cylinder length=0.012 radius=0.003
- added link right_rear_sprocket; visual cylinder length=0.004 radius=0.028; visual cylinder length=0.004 radius=0.028
- added link standoff_fl; visual cylinder length=0.030 radius=0.004
- added link standoff_fr; visual cylinder length=0.030 radius=0.004
- added link standoff_rl; visual cylinder length=0.030 radius=0.004
- added link standoff_rr; visual cylinder length=0.030 radius=0.004
- link base_link: mass 5.0 -> 2.0; geometry collision box size=0.185 0.100 0.030; visual box size=0.185 0.100 0.030
- link left_track: mass None -> 0.5; geometry collision box size=0.185 0.040 0.057; visual box size=0.130 0.038 0.006
- link right_track: mass None -> 0.5; geometry collision box size=0.185 0.040 0.057; visual box size=0.130 0.038 0.006
Joints:
- removed joint lidar_joint
- added joint antenna_left_joint: type fixed, parent jetson_nano_link, child antenna_left_link, origin xyz=-0.040 0.025 0.030 rpy=0 0 0
- added joint antenna_right_joint: type fixed, parent jetson_nano_link, child antenna_right_link, origin xyz=-0.040 -0.025 0.030 rpy=0 0 0
- added joint arduino_mega_joint: type fixed, parent platform_link, child arduino_mega_link, origin xyz=0.040 -0.050 0.009 rpy=0 0 0
- added joint base_footprint_joint: type fixed, parent base_footprint, child base_link, origin xyz=0 0 0.0285 rpy=0 0 0
- added joint jetson_nano_joint: type fixed, parent platform_link, child jetson_nano_link, origin xyz=-0.040 0.030 0.0265 rpy=0 0 0
- added joint left_front_sprocket_joint: type fixed, parent left_track, child left_front_sprocket, origin xyz=0.065 0 0 rpy=0 0 0
- added joint left_idler_joint: type fixed, parent left_track, child left_idler, origin xyz=0 0 -0.008 rpy=0 0 0
- added joint left_rear_sprocket_joint: type fixed, parent left_track, child left_rear_sprocket, origin xyz=-0.065 0 0 rpy=0 0 0
- added joint left_track_joint: type fixed, parent base_link, child left_track, origin xyz=0 0.070 0 rpy=0 0 0
- added joint platform_joint: type fixed, parent base_link, child platform_link, origin xyz=0 0 0.0315 rpy=0 0 0
- added joint right_front_sprocket_joint: type fixed, parent right_track, child right_front_sprocket, origin xyz=0.065 0 0 rpy=0 0 0
- added joint right_idler_joint: type fixed, parent right_track, child right_idler, origin xyz=0 0 -0.008 rpy=0 0 0
- added joint right_rear_sprocket_joint: type fixed, parent right_track, child right_rear_sprocket, origin xyz=-0.065 0 0 rpy=0 0 0
- added joint right_track_joint: type fixed, parent base_link, child right_track, origin xyz=0 -0.070 0 rpy=0 0 0
- added joint standoff_fl_joint: type fixed, parent base_link, child standoff_fl, origin xyz=0.080 0.070 0.015 rpy=0 0 0
- added joint standoff_fr_joint: type fixed, parent base_link, child standoff_fr, origin xyz=0.080 -0.070 0.015 rpy=0 0 0
- added joint standoff_rl_joint: type fixed, parent base_link, child standoff_rl, origin xyz=-0.080 0.070 0.015 rpy=0 0 0
- added joint standoff_rr_joint: type fixed, parent base_link, child standoff_rr, origin xyz=-0.080 -0.070 0.015 rpy=0 0 0
- joint left_motor_joint: child left_track -> left_motor_link; origin xyz=0 0.15 0 -> xyz=0 0.020 0 rpy=0 0 0
- joint right_motor_joint: child right_track -> right_motor_link; origin xyz=0 -0.15 0 -> xyz=0 -0.020 0 rpy=0 0 0

Commit message: Added realsense camera packages and created launch file

File: src/mark_five_description/urdf/robot.urdf (robot description, URDF)
Before this commit: robot mark_five_robot, 21 links, 20 joints
Links:
- added link camera_color_optical_frame
- added link camera_depth_optical_frame
- added link camera_link, mass 0.072; collision box size=0.025 0.090 0.025; visual box size=0.002 0.088 0.023
Joints:
- added joint camera_color_optical_joint: type fixed, parent camera_link, child camera_color_optical_frame, origin xyz=0.0125 0.010 0 rpy=-1.5708 0 -1.5708
- added joint camera_depth_optical_joint: type fixed, parent camera_link, child camera_depth_optical_frame, origin xyz=0.0125 0.035 0 rpy=-1.5708 0 -1.5708
- added joint camera_joint: type fixed, parent platform_link, child camera_link, origin xyz=0.090 0 0.030 rpy=0 -0.2618 0

Commit message: Tweak URDF, camera configs

File: src/mark_five_description/urdf/robot.urdf (robot description, URDF)
Before this commit: robot mark_five_robot, 24 links, 23 joints
Joints:
- joint camera_joint: origin xyz=0.090 0 0.030 rpy=0 -0.2618 0 -> xyz=0.135 0 0.025 rpy=0 0 0

Commit message: Added IMU code

File: src/mark_five_description/urdf/robot.urdf (robot description, URDF)
Before this commit: robot mark_five_robot, 24 links, 23 joints
Links:
- added link imu_link, mass 0.003; collision box size=0.025 0.018 0.003; visual box size=0.005 0.005 0.001
Joints:
- added joint imu_joint: type fixed, parent platform_link, child imu_link, origin xyz=0.0 0.0 0.010 rpy=0 0 0

Commit message: Updated URDF with new chassis

File: src/mark_five_description/urdf/robot.urdf (robot description, URDF)
Before this commit: robot mark_five_robot, 25 links, 24 joints
Links:
- link imu_link: geometry collision box size=0.016 0.026 0.003; visual box size=0.005 0.005 0.001
- link platform_link: geometry collision box size=0.210 0.200 0.003; visual box size=0.210 0.200 0.003
Joints:
- joint arduino_mega_joint: origin xyz=0.040 -0.050 0.009 rpy=0 0 0 -> xyz=0.040 -0.060 0.009 rpy=0 0 0
- joint camera_joint: origin xyz=0.135 0 0.025 rpy=0 0 0 -> xyz=0.130 0 0.025 rpy=0 0 0
- joint imu_joint: origin xyz=0.0 0.0 0.010 rpy=0 0 0 -> xyz=0.0 0.0 0.0465 rpy=0 0 0
- joint jetson_nano_joint: origin xyz=-0.040 0.030 0.0265 rpy=0 0 0 -> xyz=-0.055 0.040 0.0285 rpy=0 0 0
- joint standoff_fl_joint: origin xyz=0.080 0.070 0.015 rpy=0 0 0 -> xyz=0.030 0.030 0.015 rpy=0 0 0
- joint standoff_fr_joint: origin xyz=0.080 -0.070 0.015 rpy=0 0 0 -> xyz=0.030 -0.030 0.015 rpy=0 0 0
- joint standoff_rl_joint: origin xyz=-0.080 0.070 0.015 rpy=0 0 0 -> xyz=-0.030 0.030 0.015 rpy=0 0 0
- joint standoff_rr_joint: origin xyz=-0.080 -0.070 0.015 rpy=0 0 0 -> xyz=-0.030 -0.030 0.015 rpy=0 0 0

Commit message: Swapped Sabertooth with BTS7960

File: src/mark_five_description/urdf/robot.urdf (robot description, URDF)
Before this commit: robot mark_five_robot, 25 links, 24 joints
Links:
- removed link left_front_sprocket
- removed link left_idler
- removed link left_rear_sprocket
- removed link left_track
- removed link platform_link
- removed link right_front_sprocket
- removed link right_idler
- removed link right_rear_sprocket
- removed link right_track
- removed link standoff_fl
- removed link standoff_fr
- removed link standoff_rl
- removed link standoff_rr
- added link cart_frame_link, mass 3.5; collision box size=0.250 0.350 0.880; visual box size=0.003 0.330 0.006
- added link caster_fl, mass 0.05; collision sphere radius=0.020; visual sphere radius=0.020
- added link caster_fr, mass 0.05; collision sphere radius=0.020; visual sphere radius=0.020
- added link caster_rl, mass 0.05; collision sphere radius=0.020; visual sphere radius=0.020
- added link caster_rr, mass 0.05; collision sphere radius=0.020; visual sphere radius=0.020
- added link left_wheel, mass 0.3; collision cylinder length=0.030 radius=0.035; visual cylinder length=0.002 radius=0.012
- added link right_wheel, mass 0.3; collision cylinder length=0.030 radius=0.035; visual cylinder length=0.002 radius=0.012
- link arduino_mega_link: geometry collision box size=0.101 0.053 0.015; visual box size=0.012 0.010 0.008
- link base_link: mass 2.0 -> 8.0; geometry 
- link camera_link: mass 0.072 -> None; geometry 
- link imu_link: geometry collision box size=0.016 0.026 0.003; visual box size=0.005 0.005 0.001
- link left_motor_link: geometry visual box size=0.010 0.010 0.040; visual box size=0.024 0.024 0.024
- link right_motor_link: geometry visual box size=0.010 0.010 0.040; visual box size=0.024 0.024 0.024
Joints:
- removed joint left_front_sprocket_joint
- removed joint left_idler_joint
- removed joint left_rear_sprocket_joint
- removed joint left_track_joint
- removed joint platform_joint
- removed joint right_front_sprocket_joint
- removed joint right_idler_joint
- removed joint right_rear_sprocket_joint
- removed joint right_track_joint
- removed joint standoff_fl_joint
- removed joint standoff_fr_joint
- removed joint standoff_rl_joint
- removed joint standoff_rr_joint
- added joint cart_frame_joint: type fixed, parent base_link, child cart_frame_link, origin xyz=0 0 0 rpy=0 0 0
- added joint caster_fl_joint: type fixed, parent base_link, child caster_fl, origin xyz=0.110 0.155 -0.015 rpy=0 0 0
- added joint caster_fr_joint: type fixed, parent base_link, child caster_fr, origin xyz=0.110 -0.155 -0.015 rpy=0 0 0
- added joint caster_rl_joint: type fixed, parent base_link, child caster_rl, origin xyz=-0.110 0.155 -0.015 rpy=0 0 0
- added joint caster_rr_joint: type fixed, parent base_link, child caster_rr, origin xyz=-0.110 -0.155 -0.015 rpy=0 0 0
- added joint left_wheel_joint: type fixed, parent base_link, child left_wheel, origin xyz=0 0.180 0 rpy=0 0 0
- added joint right_wheel_joint: type fixed, parent base_link, child right_wheel, origin xyz=0 -0.180 0 rpy=0 0 0
- joint arduino_mega_joint: origin xyz=0.040 -0.060 0.009 rpy=0 0 0 -> xyz=0.040 -0.060 0.349 rpy=0 0 0; parent platform_link -> cart_frame_link
- joint base_footprint_joint: origin xyz=0 0 0.0285 rpy=0 0 0 -> xyz=0 0 0.035 rpy=0 0 0
- joint camera_color_optical_joint: origin xyz=0.0125 0.010 0 rpy=-1.5708 0 -1.5708 -> xyz=0 0 0 rpy=-1.5708 0 -1.5708
- joint camera_depth_optical_joint: origin xyz=0.0125 0.035 0 rpy=-1.5708 0 -1.5708 -> xyz=0 0 0 rpy=-1.5708 0 -1.5708
- joint camera_joint: origin xyz=0.130 0 0.025 rpy=0 0 0 -> xyz=0.115 0 0.610 rpy=0 0 0; parent platform_link -> cart_frame_link
- joint imu_joint: origin xyz=0.0 0.0 0.0465 rpy=0 0 0 -> xyz=0.0 0.0 0.350 rpy=0 0 0; parent platform_link -> cart_frame_link
- joint jetson_nano_joint: origin xyz=-0.055 0.040 0.0285 rpy=0 0 0 -> xyz=-0.030 0.040 0.371 rpy=0 0 0; parent platform_link -> cart_frame_link
- joint left_motor_joint: origin xyz=0 0.020 0 rpy=0 0 0 -> xyz=0 -0.030 0 rpy=0 0 0; parent base_link -> left_wheel
- joint right_motor_joint: origin xyz=0 -0.020 0 rpy=0 0 0 -> xyz=0 0.030 0 rpy=0 0 0; parent base_link -> right_wheel

Commit message: Updated URDF and integrated IMU back in

File: src/mark_five_description/urdf/robot.urdf (robot description, URDF)
Before this commit: robot mark_five_robot, 19 links, 18 joints
Links:
- link camera_link: mass None -> 0.072; geometry collision box size=0.025 0.090 0.025; visual box size=0.001 0.086 0.020
Joints:
- joint camera_joint: origin xyz=0.115 0 0.610 rpy=0 0 0 -> xyz=0.120 0.0 0.115 rpy=0 0 0
- joint imu_joint: origin xyz=0.0 0.0 0.350 rpy=0 0 0 -> xyz=0.096 0.0 0.152 rpy=0 0 0

Commit message: Updated pose values

File: src/mark_five_description/urdf/robot.urdf (robot description, URDF)
Before this commit: robot mark_five_robot, 19 links, 18 joints
Links:
- link left_wheel: geometry collision cylinder length=0.030 radius=0.0366; visual cylinder length=0.002 radius=0.012
- link right_wheel: geometry collision cylinder length=0.030 radius=0.0366; visual cylinder length=0.002 radius=0.012
Joints:
- joint base_footprint_joint: origin xyz=0 0 0.035 rpy=0 0 0 -> xyz=0 0 0.0366 rpy=0 0 0
- joint camera_joint: origin xyz=0.120 0.0 0.115 rpy=0 0 0 -> xyz=0.120 0.0 0.354 rpy=0 0 0
- joint caster_fl_joint: origin xyz=0.110 0.155 -0.015 rpy=0 0 0 -> xyz=0.110 0.155 -0.0166 rpy=0 0 0
- joint caster_fr_joint: origin xyz=0.110 -0.155 -0.015 rpy=0 0 0 -> xyz=0.110 -0.155 -0.0166 rpy=0 0 0
- joint caster_rl_joint: origin xyz=-0.110 0.155 -0.015 rpy=0 0 0 -> xyz=-0.110 0.155 -0.0166 rpy=0 0 0
- joint caster_rr_joint: origin xyz=-0.110 -0.155 -0.015 rpy=0 0 0 -> xyz=-0.110 -0.155 -0.0166 rpy=0 0 0
