Commit message: Urdf updates for lidar

File: src/mark_five_description/urdf/robot.urdf (robot description, URDF)
Before this commit: robot mark_five_robot, 19 links, 18 joints
Links:
- added link base_laser, mass 0.045; collision cylinder length=0.0348 radius=0.0193; visual cylinder length=0.0348 radius=0.0193
Joints:
- added joint lidar_joint: type fixed, parent cart_frame_link, child base_laser, origin xyz=0.120 0.0 0.188 rpy=0 0 0

Commit message: Tweaked URDF camera and lidar pose

File: src/mark_five_description/urdf/robot.urdf (robot description, URDF)
Before this commit: robot mark_five_robot, 20 links, 19 joints
Links:
- link cart_frame_link: geometry collision box size=0.450 0.356 0.766; visual mesh filename=package://mark_five_description/meshes/raskog_cart.stl scale=0.001 0.001 0.001
Joints:
- joint camera_joint: origin xyz=0.120 0.0 0.354 rpy=0 0 0 -> xyz=0.261 0.0 0.354 rpy=0 0 0
- joint caster_fl_joint: origin xyz=0.110 0.155 -0.0166 rpy=0 0 0 -> xyz=0.195 0.130 -0.0166 rpy=0 0 0
- joint caster_fr_joint: origin xyz=0.110 -0.155 -0.0166 rpy=0 0 0 -> xyz=0.195 -0.130 -0.0166 rpy=0 0 0
- joint caster_rl_joint: origin xyz=-0.110 0.155 -0.0166 rpy=0 0 0 -> xyz=-0.195 0.130 -0.0166 rpy=0 0 0
- joint caster_rr_joint: origin xyz=-0.110 -0.155 -0.0166 rpy=0 0 0 -> xyz=-0.195 -0.130 -0.0166 rpy=0 0 0
- joint imu_joint: origin xyz=0.096 0.0 0.152 rpy=0 0 0 -> xyz=0.191 0.0 0.152 rpy=0 0 0
- joint lidar_joint: origin xyz=0.120 0.0 0.188 rpy=0 0 0 -> xyz=0.245 0.0 0.188 rpy=0 0 0
